File: pcb/ScopeShuntX.kicad_pcb (KiCad board)
At the start: 2 copper layers, 18.5 x 28 mm, 12 parts, among them J1 Screw_Terminal_01x02, J2 Conn_Coaxial

Commit message: kicad 6
Routing:
- net /+: vias 22 -> 11
Other:
- net class Default removed
- board text added: "v${REVISION}"
- board text removed: "v010"
